File: Hardware/OpenBook_schematic.sch (EAGLE design)
At the start: 103 parts, among them IC1 BD5229G-TR, IC4 XC6220A331MR-G, J1 FH34SRJ-24S-0.5SH_99_, J2 SAMACSYS_PARTS_USB4110-GF-A, J3 QWIIC_RIGHT_ANGLE, J4 112A-TAAR-R03_ATTEND, Q1 20V/4.2A/52mΩ/1.4W, Q2 20V/4.2A/52mΩ/1.4W, Q3 SI1308EDL-T1-GE3, U1 W25Q512JVEIQ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

Commit message: Solved all issues. Final product.
Other:
- note added: "DMG2305UX-7"
- note added: "SD0805S020S1R0"
Changed lines of the file:
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@@
 <text x="297.18" y="55.88" size="3.81" layer="95">External NOR Flash 64MB</text>
 <text x="344.17" y="17.78" size="2.286" layer="94">Tudor Zaharia</text>
+<text x="129.54" y="96.52" size="1.778" layer="95" rot="R90">DMG2305UX-7</text>
+<text x="162.56" y="213.36" size="1.778" layer="95">SD0805S020S1R0</text>
+<text x="66.04" y="33.02" size="1.778" layer="95">SD0805S020S1R0</text>
 </plain>
 <instances>
